File: Hardware/Electronics/eagle_files/20200110_BehaviourSetup2.brd (EAGLE design)
At the start: 82.2 x 54.6 mm, 20 parts, among them Q1 IRF540, Q2 IRF540, Q3 IRF540

Commit message: changed eagle files to include 1N4004 diode in design
Parts:
- added D1: 1N4004, diode:DO41-10
- moved LED1 2.54 mm to (59.7, 47.0)
Connections:
- net +5V: now also D1.C
- net N$6: now also D1.A
Routing:
- net +5V: track 88.1 -> 97.0 mm
- net N$6: track 12.3 -> 21.2 mm
- net N$7: track 32.5 -> 30.0 mm
Changed lines of the file:
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@@
 <layer number="97" name="Info" color="7" fill="1" visible="no" active="no"/>
 <layer number="98" name="Guide" color="6" fill="1" visible="no" active="no"/>
+<layer number="99" name="SpiceOrder" color="5" fill="1" visible="no" active="no"/>
 </layers>
 <board>
@@
 <attribute name="VALUE" x="52.07" y="30.48" size="1.27" layer="27" ratio="10"/>
 </element>
-<element name="LED1" library="led" library_urn="urn:adsk.eagle:library:259" package="LED5MM" package3d_urn="urn:adsk.eagle:package:15799/2" value="" x="57.15" y="46.99" smashed="yes" rot="R180">
-<attribute name="NAME" x="53.975" y="46.4566" size="1.27" layer="25" ratio="10" rot="R180"/>
-<attribute name="POPULARITY" value="93" x="12.7" y="102.87" size="1.778" layer="27" rot="R180" display="off"/>
-<attribute name="VALUE" x="53.9496" y="48.7934" size="1.27" layer="27" ratio="10" rot="R180"/>
+<element name="LED1" library="led" library_urn="urn:adsk.eagle:library:259" package="LED5MM" package3d_urn="urn:adsk.eagle:package:15799/2" value="" x="59.69" y="46.99" smashed="yes" rot="R180">
+<attribute name="NAME" x="56.515" y="46.4566" size="1.27" layer="25" ratio="10" rot="R180"/>
+<attribute name="POPULARITY" value="93" x="15.24" y="102.87" size="1.778" layer="27" rot="R180" display="off"/>
+<attribute name="VALUE" x="56.4896" y="48.7934" size="1.27" layer="27" ratio="10" rot="R180"/>
 </element>
 <element name="Q1" library="transistor-power" library_urn="urn:adsk.eagle:library:400" package="TO220BV" package3d_urn="urn:adsk.eagle:package:29484/3" value="IRF540" x="10.16" y="38.1" smashed="yes">
@@
 <attribute name="POPULARITY" value="32" x="44.45" y="93.98" size="1.778" layer="27" rot="R180" display="off"/>
 <attribute name="VALUE" x="77.43" y="53.34" size="1.27" layer="27" ratio="10" rot="R180"/>
+</element>
+<element name="D1" library="diode" library_urn="urn:adsk.eagle:library:210" package="DO41-10" package3d_urn="urn:adsk.eagle:package:43336/1" value="1N4004" x="52.07" y="46.99" smashed="yes" rot="R270">
+<attribute name="NAME" x="53.721" y="49.022" size="1.27" layer="25" ratio="10" rot="R270"/>
+<attribute name="POPULARITY" value="82" x="52.07" y="46.99" size="1.778" layer="27" rot="R270" display="off"/>
+<attribute name="VALUE" x="49.276" y="49.022" size="1.27" layer="27" ratio="10" rot="R270"/>
 </element>
 </elements>
@@
 <wire x1="72.7075" y1="46.99" x2="74.89" y2="46.99" width="0.3048" layer="1"/>
 <wire x1="70.485" y1="44.7675" x2="72.7075" y2="46.99" width="0.3048" layer="1"/>
-<wire x1="51.435" y1="44.7675" x2="70.485" y2="44.7675" width="0.3048" layer="1"/>
-<wire x1="46.0375" y1="50.165" x2="51.435" y2="44.7675" width="0.3048" layer="1"/>
-<wire x1="31.4325" y1="50.165" x2="46.0375" y2="50.165" width="0.3048" layer="1"/>
+<wire x1="52.705" y1="44.7675" x2="70.485" y2="44.7675" width="0.3048" layer="1"/>
+<wire x1="47.3075" y1="50.165" x2="52.705" y2="44.7675" width="0.3048" layer="1"/>
+<wire x1="31.4325" y1="50.165" x2="47.3075" y2="50.165" width="0.3048" layer="1"/>
 <wire x1="27.94" y1="46.6725" x2="31.4325" y2="50.165" width="0.3048" layer="1"/>
 <wire x1="27.94" y1="46.6725" x2="27.38" y2="46.99" width="0.3048" layer="1"/>
@@
 <contactref element="X3" pad="1"/>
 <contactref element="Q3" pad="D"/>
-<wire x1="43.18" y1="45.085" x2="43.18" y2="35.56" width="0.3048" layer="1"/>
+<wire x1="43.18" y1="45.085" x2="43.18" y2="41.91" width="0.3048" layer="1"/>
+<wire x1="43.18" y1="41.91" x2="43.18" y2="35.56" width="0.3048" layer="1"/>
 <wire x1="41.275" y1="46.99" x2="43.18" y2="45.085" width="0.3048" layer="1"/>
 <wire x1="41.275" y1="46.99" x2="41.2" y2="46.99" width="0.3048" layer="1"/>
+<contactref element="D1" pad="A"/>
+<wire x1="43.18" y1="41.91" x2="52.07" y2="41.91" width="0.3048" layer="1"/>
 </signal>
 <signal name="+5V">
@@
 <wire x1="54.61" y1="7.62" x2="54.46" y2="7.62" width="0.3048" layer="1"/>
 <wire x1="70.8025" y1="7.62" x2="70.97" y2="7.62" width="0.3048" layer="1"/>
+<contactref element="D1" pad="C"/>
+<wire x1="46.3804" y1="47.2186" x2="50.5612375" y2="51.3994375" width="0.3048" layer="16"/>
+<wire x1="45.2628" y1="47.2186" x2="46.3804" y2="47.2186" width="0.3048" layer="16"/>
+<wire x1="50.5612375" y1="51.3994375" x2="52.07" y2="52.07" width="0.3048" layer="16"/>
+<wire x1="45.2628" y1="47.2186" x2="45.16" y2="46.99" width="0.3048" layer="16"/>
 </signal>
 <signal name="N$7">
 <contactref element="LED1" pad="A"/>
 <contactref element="R4" pad="2"/>
-<wire x1="66.9925" y1="46.99" x2="58.42" y2="46.99" width="0.3048" layer="1"/>
+<wire x1="66.9925" y1="46.99" x2="60.96" y2="46.99" width="0.3048" layer="1"/>
 <wire x1="69.215" y1="49.2125" x2="66.9925" y2="46.99" width="0.3048" layer="1"/>
 <wire x1="75.565" y1="49.2125" x2="69.215" y2="49.2125" width="0.3048" layer="1"/>
